File: extension-capes/x15-adaptor_a/x15_adaptor_a.sch (KiCad schematic (older format))
At the start: 67 parts, among them P1 FX18-60S-0.8SV15, P2 I2S, P3 SPI

Commit message: x15 adaptor production stage
Connections:
- no-connect marks 0 -> 2
Other:
- moved on the sheet: T1, T10, T11, T12, T12V0, T13, T14, T15, T16, T17, T18, T19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
