File: codec-board/power.sch (KiCad schematic (older format))
At the start: 46 parts, among them P201 PWR5V, U201 MCP1642B, U202 TLV1117, U203 ADP7102, U204 ADP7102

Commit message: changed page layout
Parts:
- D203, D204, D205: symbol LED -> LED-RESCUE-ctag-face-2-4
Changed lines of the file:
@@
 EESchema Schematic File Version 2
+LIBS:ctag-face-2-4-rescue
 LIBS:power
 LIBS:device
@@
 $EndComp
 $Comp
-L LED D204
+L LED-RESCUE-ctag-face-2-4 D204
 U 1 1 561E12A3
 P 2300 4800
@@
 $EndComp
 $Comp
-L LED D205
+L LED-RESCUE-ctag-face-2-4 D205
 U 1 1 561E2080
 P 2300 6550
@@
 $EndComp
 $Comp
-L LED D203
+L LED-RESCUE-ctag-face-2-4 D203
 U 1 1 561E5419
 P 1750 3050
